File: PCB/m1cha3l's pad.kicad_pcb (KiCad board)
At the start: 2 copper layers, 100 x 20 mm, 11 parts, among them J1 GND-VCC-SCL-SDA, J2 Headers for (Optional) Rotary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, SW1 SW_Push, SW2 SW_Push, SW3 SW_Push, SW4 SW_Push, U1 XIAO-RP2040-DIP

Commit message: Changed SW4 and OLED connection
Connections:
- J1 pad 3: Net-(J1-Pin_3) -> SCL
- J1 pad 4: Net-(J1-Pin_4) -> SDA
- SW4 pad 1: Net-(U1-GPIO6/SDA) -> SW4
- U1 pad 10: Net-(J1-Pin_4) -> SW4
- U1 pad 11: Net-(J1-Pin_3) -> unconnected-(U1-GPIO3/MOSI-Pad11)
- U1 pad 5: Net-(U1-GPIO6/SDA) -> SDA
- U1 pad 6: unconnected-(U1-GPIO7/SCL-Pad6) -> SCL
Routing:
- net SW4: track 0.00 -> 91.6 mm, vias 0 -> 2
- net Net-(U1-GPIO6/SDA): track 90.0 -> 0.00 mm
- net Net-(J1-Pin_3): track 17.4 -> 0.00 mm
- net SDA: track 0.00 -> 15.0 mm, vias 0 -> 1
- net Net-(J1-Pin_4): track 12.9 -> 0.00 mm
- net SCL: track 0.00 -> 11.4 mm, vias 0 -> 1
Changed lines of the file:
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@@
 	(net 1 "GND")
 	(net 2 "Net-(J1-Pin_2)")
-	(net 3 "Net-(J1-Pin_3)")
-	(net 4 "Net-(J1-Pin_4)")
+	(net 3 "SDA")
+	(net 4 "SCL")
 	(net 5 "Net-(U1-GPIO27{slash}ADC1{slash}A1)")
 	(net 6 "Net-(U1-GPIO28{slash}ADC2{slash}A2)")
 	(net 7 "Net-(U1-GPIO29{slash}ADC3{slash}A3)")
-	(net 8 "Net-(U1-GPIO6{slash}SDA)")
-	(net 9 "unconnected-(U1-GPIO7{slash}SCL-Pad6)")
+	(net 8 "SW4")
+	(net 9 "unconnected-(U1-GPIO3{slash}MOSI-Pad11)")
 	(net 10 "unconnected-(D4-DOUT-Pad2)")
 	(net 11 "+5V")
@@
 			(layers "*.Cu" "*.Mask")
 			(remove_unused_layers no)
-			(net 3 "Net-(J1-Pin_3)")
+			(net 4 "SCL")
 			(pinfunction "Pin_3")
 			(pintype "passive")
@@
 			(layers "*.Cu" "*.Mask")
 			(remove_unused_layers no)
-			(net 4 "Net-(J1-Pin_4)")
+			(net 3 "SDA")
 			(pinfunction "Pin_4")
 			(pintype "passive")
@@
 			(layers "*.Cu" "*.Mask")
 			(remove_unused_layers no)
-			(net 8 "Net-(U1-GPIO6{slash}SDA)")
+			(net 8 "SW4")
 			(pinfunction "1")
 			(pintype "passive")
@@
 			(layers "B.Cu" "B.Mask")
 			(roundrect_rratio 0.1)
-			(net 8 "Net-(U1-GPIO6{slash}SDA)")
+			(net 3 "SDA")
 			(pinfunction "GPIO6/SDA")
 			(pintype "passive")
@@
 			(layers "*.Cu" "*.Mask")
 			(remove_unused_layers no)
-			(net 8 "Net-(U1-GPIO6{slash}SDA)")
+			(net 3 "SDA")
 			(pinfunction "GPIO6/SDA")
 			(pintype "passive")
@@
 			(layers "B.Cu" "B.Mask")
 			(roundrect_rratio 0.1)
-			(net 9 "unconnected-(U1-GPIO7{slash}SCL-Pad6)")
+			(net 4 "SCL")
 			(pinfunction "GPIO7/SCL")
 			(pintype "passive")
@@
 			(layers "*.Cu" "*.Mask")
 			(remove_unused_layers no)
-			(net 9 "unconnected-(U1-GPIO7{slash}SCL-Pad6)")
+			(net 4 "SCL")
 			(pinfunction "GPIO7/SCL")
 			(pintype "passive")
@@
 			(layers "*.Cu" "*.Mask")
 			(remove_unused_layers no)
-			(net 4 "Net-(J1-Pin_4)")
+			(net 8 "SW4")
 			(pinfunction "GPIO4/MISO")
 			(pintype "passive")
@@
 			(layers "B.Cu" "B.Mask")
 			(roundrect_rratio 0.1)
-			(net 4 "Net-(J1-Pin_4)")
+			(net 8 "SW4")
 			(pinfunction "GPIO4/MISO")
 			(pintype "passive")
@@
 			(layers "*.Cu" "*.Mask")
 			(remove_unused_layers no)
-			(net 3 "Net-(J1-Pin_3)")
+			(net 9 "unconnected-(U1-GPIO3{slash}MOSI-Pad11)")
 			(pinfunction "GPIO3/MOSI")
 			(pintype "passive")
@@
 			(layers "B.Cu" "B.Mask")
 			(roundrect_rratio 0.1)
-			(net 3 "Net-(J1-Pin_3)")
+			(net 9 "unconnected-(U1-GPIO3{slash}MOSI-Pad11)")
 			(pinfunction "GPIO3/MOSI")
 			(pintype "passive")
@@
 	)
 	(segment
-		(start 116.84 107)
-		(end 123.84 107)
+		(start 125 105.7)
+		(end 125 105)
 		(width 0.2)
 		(layer "F.Cu")
@@
 	)
 	(segment
-		(start 123.84 107)
-		(end 124.84 106)
+		(start 127.84 108.54)
+		(end 125 105.7)
 		(width 0.2)
 		(layer "F.Cu")
 		(net 3)
 	)
-	(segment
-		(start 116 112.62)
-		(end 116.22 112.4)
-		(width 0.2)
-		(layer "F.Cu")
+	(via
+		(at 125 105)
+		(size 0.6)
+		(drill 0.3)
+		(layers "F.Cu" "B.Cu")
 		(net 3)
 	)
 	(segment
-		(start 116.22 107.62)
-		(end 116.84 107)
+		(start 125 105)
+		(end 118.54 98.54)
 		(width 0.2)
-		(layer "F.Cu")
+		(layer "B.Cu")
 		(net 3)
 	)
 	(segment
-		(start 116.22 112.4)
-		(end 116.22 107.62)
+		(start 118.54 98.54)
+		(end 118.54 97.38)
 		(width 0.2)
-		(layer "F.Cu")
+		(layer "B.Cu")
 		(net 3)
 	)
 	(segment
-		(start 124.84 106)
-		(end 127.84 106)
+		(start 127.84 106)
+		(end 126 104.16)
 		(width 0.2)
 		(layer "F.Cu")
-		(net 3)
+		(net 4)
 	)
 	(segment
-		(start 119.3 108.54)
-		(end 127.84 108.54)
+		(start 126 104.16)
+		(end 126 104.06)
 		(width 0.2)
 		(layer "F.Cu")
 		(net 4)
 	)
+	(via
+		(at 126 104.06)
+		(size 0.6)
+		(drill 0.3)
+		(layers "F.Cu" "B.Cu")
+		(net 4)
+	)
 	(segment
-		(start 118.54 112.62)
-		(end 118.76 112.4)
+		(start 121.08 99.08)
+		(end 121.08 97.38)
 		(width 0.2)
-		(layer "F.Cu")
+		(layer "B.Cu")
 		(net 4)
 	)
 	(segment
-		(start 118.76 109.08)
-		(end 119.3 108.54)
+		(start 126 104)
+		(end 121.08 99.08)
 		(width 0.2)
-		(layer "F.Cu")
+		(layer "B.Cu")
 		(net 4)
 	)
 	(segment
-		(start 118.76 112.4)
-		(end 118.76 109.08)
+		(start 126 104.06)
+		(end 126 104)
 		(width 0.2)
-		(layer "F.Cu")
+		(layer "B.Cu")
 		(net 4)
 	)
@@
 	)
 	(segment
+		(start 119.236 104)
+		(end 119.197 104)
+		(width 0.2)
+		(layer "F.Cu")
+		(net 8)
+	)
+	(segment
+		(start 124.439 100.8339)
+		(end 121.2729 104)
+		(width 0.2)
+		(layer "F.Cu")
+		(net 8)
+	)
+	(segment
+		(start 124.439 99.6997)
+		(end 124.439 100.8339)
+		(width 0.2)
+		(layer "F.Cu")
+		(net 8)
+	)
+	(segment
 		(start 126.4217 97.717)
 		(end 124.439 99.6997)
@@
 	)
 	(segment
-		(start 178.7441 97.717)
-		(end 126.4217 97.717)
+		(start 119.197 104)
+		(end 119 104.197)
 		(width 0.2)
 		(layer "F.Cu")
@@
 	)
 	(segment
-		(start 197.38 99.92)
-		(end 195.46 98)
+		(start 118 109)
+		(end 118 112.08)
+		(width 0.2)
+		(layer "F.Cu")
+		(net 8)
+	)
+	(segment
+		(start 118 112.08)
+		(end 118.25645 112.33645)
 		(width 0.2)
 		(layer "F.Cu")
@@
 	)
 	(segment
-		(start 179.0271 98)
-		(end 178.7441 97.717)
+		(start 197.38 99.92)
+		(end 195.46 98)
 		(width 0.2)
 		(layer "F.Cu")
@@
 	)
 	(segment
-		(start 118.76 104.316)
-		(end 118.76 97.6)
+		(start 121.2729 104)
+		(end 119.236 104)
 		(width 0.2)
 		(layer "F.Cu")
@@
 	)
 	(segment
-		(start 118.76 97.6)
-		(end 118.54 97.38)
+		(start 119 108)
+		(end 118 109)
 		(width 0.2)
 		(layer "F.Cu")
@@
 	)
 	(segment
-		(start 124.439 99.6997)
-		(end 124.439 100.8339)
+		(start 179.0271 98)
+		(end 178.7441 97.717)
 		(width 0.2)
 		(layer "F.Cu")
@@
 	)
 	(segment
-		(start 120.8769 104.396)
-		(end 118.84 104.396)
+		(start 178.7441 97.717)
+		(end 126.4217 97.717)
 		(width 0.2)
 		(layer "F.Cu")
@@
 	)
 	(segment
-		(start 124.439 100.8339)
-		(end 120.8769 104.396)
+		(start 118.54 112.62)
+		(end 118.76 112.4)
 		(width 0.2)
 		(layer "F.Cu")
 		(net 8)
 	)
+	(via
+		(at 119 104.197)
+		(size 0.6)
+		(drill 0.3)
+		(layers "F.Cu" "B.Cu")
+		(net 8)
+	)
+	(via
+		(at 119 108)
+		(size 0.6)
+		(drill 0.3)
+		(layers "F.Cu" "B.Cu")
+		(net 8)
+	)
 	(segment
-		(start 118.84 104.396)
-		(end 118.76 104.316)
+		(start 119 104.197)
+		(end 119 108)
 		(width 0.2)
-		(layer "F.Cu")
+		(layer "B.Cu")
 		(net 8)
 	)
 	(segment
+		(start 116 112.62)
+		(end 116.22 112.4)
+		(width 0.2)
+		(layer "F.Cu")
+		(net 9)
+	)
+	(segment
